Commit message: feat(launch): Add launch file python and xml to bringup robot

File: src/my_robot_description/urdf/ar_base.xacro (robot description, xacro)
@@ -9,8 +9,14 @@
         <visual>
             <geometry>
-                <mesh filename="package://my_robot_description/meshes/base_link.STL"/>
+                <mesh filename="package://my_robot_description/meshes/visuals/base_link.STL"/>
             </geometry>
             <origin xyz="0 0 0" rpy="0 0 0"/>
         </visual>
+        <collision>
+            <geometry>
+                <mesh filename="package://my_robot_description/meshes/collisions/base_link.STL"/>
+            </geometry>
+            <origin xyz="0 0 0" rpy="0 0 0"/>
+        </collision>
     </link>
     <joint name = "Base_joint" type ="fixed">
@@ -23,7 +29,13 @@
             <origin rpy="0 0 0" xyz="0 0 0"/>
             <geometry>
-                <mesh filename="package://my_robot_description/meshes/link_1.STL"/>
+                <mesh filename="package://my_robot_description/meshes/visuals/link_1.STL"/>
             </geometry>
         </visual>
+        <collision>
+            <origin rpy="0 0 0" xyz="0 0 0"/>
+            <geometry>
+                <mesh filename="package://my_robot_description/meshes/collisions/link_1.STL"/>
+            </geometry>
+        </collision>
     </link>
     <joint name="Arm_joint1" type="revolute">
@@ -38,7 +50,13 @@
             <origin rpy="0 0 0" xyz="0 0 0"/>
             <geometry>
-                <mesh filename="package://my_robot_description/meshes/link_2.STL"/>
+                <mesh filename="package://my_robot_description/meshes/visuals/link_2.STL"/>
             </geometry>
         </visual>
+        <collision>
+            <origin rpy="0 0 0" xyz="0 0 0"/>
+            <geometry>
+                <mesh filename="package://my_robot_description/meshes/collisions/link_2.STL"/>
+            </geometry>
+        </collision>
     </link>
     <joint name="Arm_joint2" type="revolute">
@@ -53,7 +71,13 @@
             <origin rpy="0 0 0" xyz="0 0 0"/>
             <geometry>
-                <mesh filename="package://my_robot_description/meshes/link_3.STL"/>
+                <mesh filename="package://my_robot_description/meshes/visuals/link_3.STL"/>
             </geometry>
         </visual>
+        <collision>
+            <origin rpy="0 0 0" xyz="0 0 0"/>
+            <geometry>
+                <mesh filename="package://my_robot_description/meshes/collisions/link_3.STL"/>
+            </geometry>
+        </collision>
     </link>
     <joint name="Arm_joint3" type="revolute">
@@ -68,7 +92,13 @@
             <origin rpy="0 0 0" xyz="0 0 0"/>
             <geometry>
-                <mesh filename="package://my_robot_description/meshes/link_4.STL"/>
+                <mesh filename="package://my_robot_description/meshes/visuals/link_4.STL"/>
             </geometry>
         </visual>
+        <collision>
+            <origin rpy="0 0 0" xyz="0 0 0"/>
+            <geometry>
+                <mesh filename="package://my_robot_description/meshes/collisions/link_4.STL"/>
+            </geometry>
+        </collision>
     </link>
     <joint name="Arm_joint4" type="revolute">
@@ -83,7 +113,13 @@
             <origin rpy="0 0 0" xyz="0 0 0"/>
             <geometry>
-                <mesh filename="package://my_robot_description/meshes/link_5.STL"/>
+                <mesh filename="package://my_robot_description/meshes/visuals/link_5.STL"/>
             </geometry>
         </visual>
+        <collision>
+            <origin rpy="0 0 0" xyz="0 0 0"/>
+            <geometry>
+                <mesh filename="package://my_robot_description/meshes/collisions/link_5.STL"/>
+            </geometry>
+        </collision>
     </link>
     <joint name="Arm_joint5" type="revolute">
@@ -98,7 +134,13 @@
             <origin rpy="0 0 0" xyz="0 0 0"/>
             <geometry>
-                <mesh filename="package://my_robot_description/meshes/link_6.STL"/>
+                <mesh filename="package://my_robot_description/meshes/visuals/link_6.STL"/>
             </geometry>
         </visual>
+        <collision>
+            <origin rpy="0 0 0" xyz="0 0 0"/>
+            <geometry>
+                <mesh filename="package://my_robot_description/meshes/collisions/link_6.STL"/>
+            </geometry>
+        </collision>
     </link>
     <joint name="Arm_joint6" type="revolute">

Commit message: feat(moveit): Add moveit

File: src/my_robot_description/urdf/ar_base.xacro (robot description, xacro)
@@ -26,4 +26,9 @@
     </joint>
     <link name="Arm_link1">
+        <inertial>
+        <origin rpy="0 0 0" xyz="-0.022706 0.04294 -0.12205"/>
+        <mass value="0.88065"/>
+        <inertia ixx="0.0034" ixy="0.00042296" ixz="-0.00089231" iyy="0.0041778" iyz="0.0010848" izz="0.0027077"/>
+        </inertial>
         <visual>
             <origin rpy="0 0 0" xyz="0 0 0"/>
@@ -47,4 +52,9 @@
     </joint>
     <link name="Arm_link2">
+        <inertial>
+        <origin rpy="0 0 0" xyz="0.064818 -0.11189 -0.038671"/>
+        <mass value="0.57738"/>
+        <inertia ixx="0.0047312" ixy="0.0022624" ixz="0.00032144" iyy="0.0020836" iyz="-0.00056569" izz="0.0056129"/>
+        </inertial>
         <visual>
             <origin rpy="0 0 0" xyz="0 0 0"/>
@@ -68,4 +78,9 @@
     </joint>
     <link name="Arm_link3">
+        <inertial>
+        <origin rpy="0 0 0" xyz="-0.00029765 -0.023661 -0.0019125"/>
+        <mass value="0.1787"/>
+        <inertia ixx="0.0001685" ixy="-2.7713E-05" ixz="5.6885E-06" iyy="0.00012865" iyz="2.9256E-05" izz="0.00020744"/>
+        </inertial>
         <visual>
             <origin rpy="0 0 0" xyz="0 0 0"/>
@@ -89,4 +104,9 @@
     </joint>
     <link name="Arm_link4">
+        <inertial>
+        <origin rpy="0 0 0" xyz="-0.0016798 -0.00057319 -0.074404"/>
+        <mass value="0.34936"/>
+        <inertia ixx="0.0030532" ixy="-1.8615E-05" ixz="-7.0047E-05" iyy="0.0031033" iyz="-2.3301E-05" izz="0.00022264"/>
+        </inertial>
         <visual>
             <origin rpy="0 0 0" xyz="0 0 0"/>
@@ -110,4 +130,9 @@
     </joint>
     <link name="Arm_link5">
+        <inertial>
+        <origin rpy="0 0 0" xyz="0.0015066 -1.3102E-05 -0.012585"/>
+        <mass value="0.11562"/>
+        <inertia ixx="5.5035E-05" ixy="-1.019E-08" ixz="-2.6243E-06" iyy="8.2921E-05" iyz="1.4437E-08" izz="5.2518E-05"/>
+        </inertial>
         <visual>
             <origin rpy="0 0 0" xyz="0 0 0"/>
@@ -131,4 +156,9 @@
     </joint>
     <link name="Arm_endlink">
+        <inertial>
+        <origin rpy="0 0 0" xyz="2.9287E-10 -1.6472E-09 0.0091432"/>
+        <mass value="0.013863"/>
+        <inertia ixx="1.3596E-06" ixy="3.0585E-13" ixz="5.7102E-14" iyy="1.7157E-06" iyz="6.3369E-09" izz="2.4332E-06"/>
+        </inertial>
         <visual>
             <origin rpy="0 0 0" xyz="0 0 0"/>
